File: Fan.sch (KiCad schematic (older format))
At the start: 9 parts, among them Q2 MOSFET_N, Q3 MOSFET_N, Q4 MOSFET_N, U20 OPA4170, U6 MCP4922-E/P

Commit message: Power Modification Module
Parts:
- removed Q3, Q4: MOSFET_N, ~, symbol MOSFET_N
- removed U6: MCP4922-E/P, DIP14, symbol MCP4922-E/P
- added C12, C13: C, ~, symbol C
- added Q3, Q4: AOD476, ~, symbol MOS_N_NUM
- added U4: MCP4801, symbol MCP4801
- D5: value DIODE -> B130-13-F; MFG Name (none) -> Diodes Inc; MFG Part Number (none) -> B130-13-F
- Q2: value MOSFET_N -> DMN65D8L-7; MFG Name (none) -> Diodes Inc; MFG Part Number (none) -> DMN65D8L-7
- TH5: value THERMISTOR -> MINISMDC050F-2; MFG Name (none) -> TE Connectivity; MFG Part Number (none) -> MINISMDC050F-2
Connections:
- net +12C: now also C13.1
- net AGND: now also C12.1, C13.2, Q3.3 (S), U4.7 (Vss)
- net CS_N: now also U4.2 (~CS)
- net CURR_MEAS: now also Q3.2 (D), Q4.3 (S)
- net FAN_MODE: now also Q3.1 (G)
- net FAN_OUT-: now also Q4.2 (D)
- net MOSI: now also U4.4 (SDI)
- net SCLK: now also U4.3 (SCK)
- net at U20.14: now also Q4.1 (G)
- net at R17.1: now also U4.8 (Vout)
- new net +5V: C12.2, U4.1 (Vdd)
- new net ~LDAC: U4.5 (~LDAC)
- new net ~SHDN: U4.6 (~SHDN)
Other:
- note added: "SHOULD THIS BE A DIFFERENT GROUND?"
Changed lines of the file:
@@
 Sheet 5 9
 Title ""
-Date "17 oct 2013"
+Date "27 oct 2013"
 Rev ""
 Comp ""
@@
 Comment4 ""
 $EndDescr
-Text HLabel 2600 2950 0    60   Input ~ 0
+Text HLabel 2600 3100 0    60   Input ~ 0
 FAN_PWM
 Text HLabel 2600 4450 0    60   Output ~ 0
@@
 	1    0    0    -1
 $EndComp
-$Comp
-L MOSFET_N Q4
-U 1 1 523BC5BC
-P 7500 2150
-F 0 "Q4" H 7510 2320 60  0000 R CNN
-F 1 "MOSFET_N" H 7510 2000 60  0000 R CNN
-F 2 "~" H 7500 2150 60  0000 C CNN
-F 3 "~" H 7500 2150 60  0000 C CNN
-	1    7500 2150
-	1    0    0    -1
-$EndComp
 Wire Wire Line
 	6550 2150 7300 2150
@@
 $EndComp
 $Comp
-L AGND #PWR036
+L AGND #PWR45
 U 1 1 523BC6A2
 P 7600 4250
-F 0 "#PWR036" H 7600 4250 40  0001 C CNN
+F 0 "#PWR45" H 7600 4250 40  0001 C CNN
 F 1 "AGND" H 7600 4180 50  0000 C CNN
 F 2 "" H 7600 4250 60  0000 C CNN
@@
 	7600 3950 7600 4250
 $Comp
-L +12V #PWR037
+L +12V #PWR42
 U 1 1 523BC6C6
 P 5950 1600
-F 0 "#PWR037" H 5950 1550 20  0001 C CNN
+F 0 "#PWR42" H 5950 1550 20  0001 C CNN
 F 1 "+12V" H 5950 1700 30  0000 C CNN
 F 2 "" H 5950 1600 60  0000 C CNN
@@
 $EndComp
 $Comp
-L -12V #PWR038
+L -12V #PWR43
 U 1 1 523BC6E4
 P 5950 2850
-F 0 "#PWR038" H 5950 2980 20  0001 C CNN
+F 0 "#PWR43" H 5950 2980 20  0001 C CNN
 F 1 "-12V" H 5950 2950 30  0000 C CNN
 F 2 "" H 5950 2850 60  0000 C CNN
@@
 	4250 2750 4250 2950
 $Comp
-L AGND #PWR039
+L AGND #PWR41
 U 1 1 523BC839
 P 4250 3000
-F 0 "#PWR039" H 4250 3000 40  0001 C CNN
+F 0 "#PWR41" H 4250 3000 40  0001 C CNN
 F 1 "AGND" H 4250 2930 50  0000 C CNN
 F 2 "" H 4250 3000 60  0000 C CNN
@@
 	1    0    0    -1
 $EndComp
-$Comp
-L MCP4922-E/P U6
-U 1 1 523BC8D3
-P 3100 2200
-F 0 "U6" H 3250 2600 40  0000 L BNN
-F 1 "MCP4922-E/P" H 3250 2550 40  0000 L BNN
-F 2 "DIP14" H 3100 2200 30  0000 C CIN
-F 3 "" H 3100 2200 60  0000 C CNN
-	1    3100 2200
-	1    0    0    -1
-$EndComp
 Text HLabel 2600 3200 0    60   Output ~ 0
 CURR_MEAS
 Connection ~ 5350 3200
 Wire Wire Line
-	2600 2950 3600 2950
+	2600 3100 3600 3100
 $Comp
 L R R17
@@
 $EndComp
 Wire Wire Line
-	3650 2050 3650 2050
-Text HLabel 2200 2000 0    60   Input ~ 0
+	3550 2050 3650 2050
+Text HLabel 1600 2000 0    60   Input ~ 0
 MOSI
-Text HLabel 2200 2300 0    60   Input ~ 0
-MISO
-Text HLabel 2200 2200 0    60   Input ~ 0
+Text HLabel 1600 1700 0    60   Input ~ 0
 CS_N
-Text HLabel 2200 2100 0    60   Input ~ 0
+Text HLabel 1600 1850 0    60   Input ~ 0
 SCLK
-Wire Wire Line
-	2200 2000 2550 2000
-Wire Wire Line
-	2200 2100 2550 2100
-Wire Wire Line
-	2200 2200 2550 2200
-$Comp
-L MOSFET_N Q3
-U 1 1 52492E73
-P 7250 3550
-F 0 "Q3" H 7260 3720 60  0000 R CNN
-F 1 "MOSFET_N" H 7260 3400 60  0000 R CNN
-F 2 "~" H 7250 3550 60  0000 C CNN
-F 3 "~" H 7250 3550 60  0000 C CNN
-	1    7250 3550
-	1    0    0    -1
-$EndComp
 $Comp
 L THERMISTOR TH5
@@
 P 7600 1150
 F 0 "TH5" V 7700 1200 50  0000 C CNN
-F 1 "THERMISTOR" V 7500 1150 50  0000 C CNN
+F 1 "MINISMDC050F-2" V 7500 1150 50  0000 C CNN
 F 2 "~" H 7600 1150 60  0000 C CNN
 F 3 "~" H 7600 1150 60  0000 C CNN
+F 4 "TE Connectivity" H 7600 1150 60  0001 C CNN "MFG Name"
+F 5 "MINISMDC050F-2" H 7600 1150 60  0001 C CNN "MFG Part Number"
 	1    7600 1150
 	1    0    0    -1
@@
 P 7200 1550
 F 0 "D5" H 7200 1650 40  0000 C CNN
-F 1 "DIODE" H 7200 1450 40  0000 C CNN
+F 1 "B130-13-F" H 7200 1450 40  0000 C CNN
 F 2 "~" H 7200 1550 60  0000 C CNN
 F 3 "~" H 7200 1550 60  0000 C CNN
+F 4 "Diodes Inc" H 7200 1550 60  0001 C CNN "MFG Name"
+F 5 "B130-13-F" H 7200 1550 60  0001 C CNN "MFG Part Number"
 	1    7200 1550
 	0    -1   -1   0
@@
 P 4150 2550
 F 0 "Q2" H 4160 2720 60  0000 R CNN
-F 1 "MOSFET_N" H 4160 2400 60  0000 R CNN
+F 1 "DMN65D8L-7" H 4160 2400 60  0000 R CNN
 F 2 "~" H 4150 2550 60  0000 C CNN
 F 3 "~" H 4150 2550 60  0000 C CNN
+F 4 "Diodes Inc" H 4150 2550 60  0001 C CNN "MFG Name"
+F 5 "DMN65D8L-7" H 4150 2550 60  0001 C CNN "MFG Part Number"
 	1    4150 2550
 	1    0    0    -1
@@
 Connection ~ 4250 2050
 Wire Wire Line
-	3600 2950 3600 2550
+	3600 3100 3600 2550
 Wire Wire Line
 	3600 2550 3950 2550
@@
 	7050 3550 2600 3550
 $Comp
-L +12C #PWR040
+L +12C #PWR44
 U 1 1 52493C3F
 P 7600 750
-F 0 "#PWR040" H 7600 720 30  0001 C CNN
+F 0 "#PWR44" H 7600 720 30  0001 C CNN
 F 1 "+12C" H 7600 860 40  0000 C CNN
 F 2 "" H 7600 750 60  0000 C CNN
@@
 Wire Wire Line
 	5950 1750 5950 1600
+$Comp
+L MCP4801 U4
+U 1 1 52642E1E
+P 2700 1950
+F 0 "U4" H 2800 1350 60  0000 C CNN
+F 1 "MCP4801" H 2650 1850 60  0000 C CNN
+F 2 "" H 2700 1950 60  0000 C CNN
+F 3 "" H 2700 1950 60  0000 C CNN
+	1    2700 1950
+	1    0    0    -1
+$EndComp
+Wire Wire Line
+	1600 1700 1800 1700
+Wire Wire Line
+	1800 1850 1600 1850
+Wire Wire Line
+	1600 2000 1800 2000
+Text HLabel 1600 2150 0    60   Input ~ 0
+~LDAC
+Text HLabel 1600 2300 0    60   Input ~ 0
+~SHDN
+Wire Wire Line
+	1600 2150 1800 2150
+Wire Wire Line
+	1800 2300 1600 2300
+$Comp
+L +5V #PWR39
+U 1 1 526E3891
+P 2550 950
+F 0 "#PWR39" H 2550 1040 20  0001 C CNN
+F 1 "+5V" H 2550 1040 30  0000 C CNN
+F 2 "" H 2550 950 60  0000 C CNN
+F 3 "" H 2550 950 60  0000 C CNN
+	1    2550 950
+	1    0    0    -1
+$EndComp
+Wire Wire Line
+	2550 950  2550 1300
+$Comp
+L C C12
+U 1 1 526E38C9
+P 2300 1100
+F 0 "C12" H 2300 1200 40  0000 L CNN
+F 1 "C" H 2306 1015 40  0000 L CNN
+F 2 "~" H 2338 950 30  0000 C CNN
+F 3 "~" H 2300 1100 60  0000 C CNN
+	1    2300 1100
+	0    -1   -1   0
+$EndComp
+$Comp
+L AGND #PWR38
+U 1 1 526E38D8
+P 2000 1250
+F 0 "#PWR38" H 2000 1250 40  0001 C CNN
+F 1 "AGND" H 2000 1180 50  0000 C CNN
+F 2 "" H 2000 1250 60  0000 C CNN
+F 3 "" H 2000 1250 60  0000 C CNN
+	1    2000 1250
+	1    0    0    -1
+$EndComp
+Wire Wire Line
+	2000 1250 2000 1100
+Wire Wire Line
+	2000 1100 2100 1100
+Wire Wire Line
+	2500 1100 2550 1100
+Connection ~ 2550 1100
+$Comp
+L AGND #PWR40
+U 1 1 526E399E
+P 2550 2850
+F 0 "#PWR40" H 2550 2850 40  0001 C CNN
+F 1 "AGND" H 2550 2780 50  0000 C CNN
+F 2 "" H 2550 2850 60  0000 C CNN
+F 3 "" H 2550 2850 60  0000 C CNN
+	1    2550 2850
+	1    0    0    -1
+$EndComp
+Wire Wire Line
+	2550 2850 2550 2750
+$Comp
+L C C13
+U 1 1 526E46C7
+P 8300 850
+F 0 "C13" H 8300 950 40  0000 L CNN
+F 1 "C" H 8306 765 40  0000 L CNN
+F 2 "~" H 8338 700 30  0000 C CNN
+F 3 "~" H 8300 850 60  0000 C CNN
+	1    8300 850
+	0    -1   -1   0
+$EndComp
+$Comp
+L AGND #PWR46
+U 1 1 526E46CF
+P 8600 1100
+F 0 "#PWR46" H 8600 1100 40  0001 C CNN
+F 1 "AGND" H 8600 1030 50  0000 C CNN
+F 2 "" H 8600 1100 60  0000 C CNN
+F 3 "" H 8600 1100 60  0000 C CNN
+	1    8600 1100
+	1    0    0    -1
+$EndComp
+Wire Wire Line
+	8600 1100 8600 850
+Wire Wire Line
+	8600 850  8500 850
+Wire Wire Line
+	8100 850  7600 850
+Connection ~ 7600 850
+Text Notes 8800 1200 0    60   ~ 0
+SHOULD THIS BE A DIFFERENT GROUND?
+Text Notes 7750 4350 0    60   ~ 0
+SHOULD THIS BE A DIFFERENT GROUND?
+$Comp
+L MOS_N_NUM Q4
+U 1 1 526E489B
+P 7500 2150
+F 0 "Q4" H 7510 2320 60  0000 R CNN
+F 1 "AOD476" H 7510 2000 60  0000 R CNN
+F 2 "~" H 7500 2150 60  0000 C CNN
+F 3 "~" H 7500 2150 60  0000 C CNN
+F 4 "Alpha and Omega" H 7500 2150 60  0001 C CNN "MFG Name"
+F 5 "AOD476" H 7500 2150 60  0001 C CNN "MFG Part Number"
+	1    7500 2150
+	1    0    0    -1
+$EndComp
+$Comp
+L MOS_N_NUM Q3
+U 1 1 526E48ED
+P 7250 3550
+F 0 "Q3" H 7260 3720 60  0000 R CNN
+F 1 "AOD476" H 7260 3400 60  0000 R CNN
+F 2 "~" H 7250 3550 60  0000 C CNN
+F 3 "~" H 7250 3550 60  0000 C CNN
+F 4 "Alpha and Omega" H 7250 3550 60  0001 C CNN "MFG Name"
+F 5 "AOD476" H 7250 3550 60  0001 C CNN "MFG Part Number"
+	1    7250 3550
+	1    0    0    -1
+$EndComp
 $EndSCHEMATC
