File: Power.sch (KiCad schematic (older format))
At the start: 13 parts, among them P1 24 Pin MiniFit JR, SW1 SWITCH_INV

Commit message: Power Modification Module
Parts:
- L1, L2, L4: value INDUCTOR -> CM322522-220KL; MFG Name (none) -> Bourns Inc; MFG Part Number (none) -> CM322522-220KL
- SW1: value SWITCH_INV -> OS102011MA1QN1; MFG Name (none) -> C&C Components; MFG Part Number (none) -> OS102011MA1QN1
- TH1, TH2, TH3, TH4: value THERMISTOR -> MINISMDC050F-2; MFG Name (none) -> TE Connectivity; MFG Part Number (none) -> MINISMDC050F-2
Changed lines of the file:
@@
 Sheet 3 9
 Title ""
-Date "17 oct 2013"
+Date "27 oct 2013"
 Rev ""
 Comp ""
@@
 	4100 1950 4100 1250
 $Comp
-L +12P #PWR018
+L +12P #PWR23
 U 1 1 523E6AD9
 P 4100 1250
-F 0 "#PWR018" H 4100 1220 30  0001 C CNN
+F 0 "#PWR23" H 4100 1220 30  0001 C CNN
 F 1 "+12P" H 4100 1350 30  0000 C CNN
 F 2 "" H 4100 1250 60  0000 C CNN
@@
 P 3000 2650
 F 0 "SW1" H 2800 2800 50  0000 C CNN
-F 1 "SWITCH_INV" H 2850 2500 50  0000 C CNN
+F 1 "OS102011MA1QN1" H 2850 2500 50  0000 C CNN
 F 2 "~" H 3000 2650 60  0000 C CNN
 F 3 "~" H 3000 2650 60  0000 C CNN
+F 4 "C&C Components" H 3000 2650 60  0001 C CNN "MFG Name"
+F 5 "OS102011MA1QN1" H 3000 2650 60  0001 C CNN "MFG Part Number"
 	1    3000 2650
 	1    0    0    -1
 $EndComp
 $Comp
-L -12P #PWR019
+L -12P #PWR25
 U 1 1 523E6B53
 P 4500 1250
-F 0 "#PWR019" H 4500 1380 20  0001 C CNN
+F 0 "#PWR25" H 4500 1380 20  0001 C CNN
 F 1 "-12P" H 4500 1350 30  0000 C CNN
 F 2 "" H 4500 1250 60  0000 C CNN
@@
 Connection ~ 1450 1750
 $Comp
-L GND #PWR020
+L GND #PWR18
 U 1 1 523E6D4C
 P 900 1900
-F 0 "#PWR020" H 900 1900 30  0001 C CNN
+F 0 "#PWR18" H 900 1900 30  0001 C CNN
 F 1 "GND" H 900 1830 30  0001 C CNN
 F 2 "" H 900 1900 60  0000 C CNN
@@
 	3650 2750 3650 2900
 $Comp
-L GND #PWR021
+L GND #PWR21
 U 1 1 523E6DB4
 P 3650 2900
-F 0 "#PWR021" H 3650 2900 30  0001 C CNN
+F 0 "#PWR21" H 3650 2900 30  0001 C CNN
 F 1 "GND" H 3650 2830 30  0001 C CNN
 F 2 "" H 3650 2900 60  0000 C CNN
@@
 $EndComp
 $Comp
-L +3.3V #PWR022
+L +3.3V #PWR24
 U 1 1 523E6DF4
 P 4150 2500
-F 0 "#PWR022" H 4150 2460 30  0001 C CNN
+F 0 "#PWR24" H 4150 2460 30  0001 C CNN
 F 1 "+3.3V" H 4150 2610 30  0000 C CNN
 F 2 "" H 4150 2500 60  0000 C CNN
@@
 	4150 2550 4150 2500
 $Comp
-L +12P #PWR023
+L +12P #PWR27
 U 1 1 523E7000
 P 5400 2050
-F 0 "#PWR023" H 5400 2020 30  0001 C CNN
+F 0 "#PWR27" H 5400 2020 30  0001 C CNN
 F 1 "+12P" H 5400 2150 30  0000 C CNN
 F 2 "" H 5400 2050 60  0000 C CNN
@@
 $EndComp
 $Comp
-L GND #PWR024
+L GND #PWR29
 U 1 1 523E701E
 P 6050 2600
-F 0 "#PWR024" H 6050 2600 30  0001 C CNN
+F 0 "#PWR29" H 6050 2600 30  0001 C CNN
 F 1 "GND" H 6050 2530 30  0001 C CNN
 F 2 "" H 6050 2600 60  0000 C CNN
@@
 $EndComp
 $Comp
-L INDUCTOR L1
-U 1 1 523E702D
-P 5950 2050
-F 0 "L1" V 5900 2050 40  0000 C CNN
-F 1 "INDUCTOR" V 6050 2050 40  0000 C CNN
-F 2 "~" H 5950 2050 60  0000 C CNN
-F 3 "~" H 5950 2050 60  0000 C CNN
-	1    5950 2050
-	0    -1   -1   0
-$EndComp
-$Comp
-L INDUCTOR L2
-U 1 1 523E703A
-P 5950 3150
-F 0 "L2" V 5900 3150 40  0000 C CNN
-F 1 "INDUCTOR" V 6050 3150 40  0000 C CNN
-F 2 "~" H 5950 3150 60  0000 C CNN
-F 3 "~" H 5950 3150 60  0000 C CNN
-	1    5950 3150
-	0    -1   -1   0
-$EndComp
-$Comp
-L -12P #PWR025
+L -12P #PWR28
 U 1 1 523E7201
 P 5400 3150
-F 0 "#PWR025" H 5400 3280 20  0001 C CNN
+F 0 "#PWR28" H 5400 3280 20  0001 C CNN
 F 1 "-12P" H 5400 3250 30  0000 C CNN
 F 2 "" H 5400 3150 60  0000 C CNN
@@
 	5650 3150 5400 3150
 $Comp
-L -12V #PWR026
+L -12V #PWR33
 U 1 1 523E7358
 P 6850 3150
-F 0 "#PWR026" H 6850 3280 20  0001 C CNN
+F 0 "#PWR33" H 6850 3280 20  0001 C CNN
 F 1 "-12V" H 6850 3250 30  0000 C CNN
 F 2 "" H 6850 3150 60  0000 C CNN
@@
 $EndComp
 $Comp
-L +12V #PWR027
+L +12V #PWR32
 U 1 1 523E7367
 P 6850 2050
-F 0 "#PWR027" H 6850 2000 20  0001 C CNN
+F 0 "#PWR32" H 6850 2000 20  0001 C CNN
 F 1 "+12V" H 6850 2150 30  0000 C CNN
 F 2 "" H 6850 2050 60  0000 C CNN
@@
 Connection ~ 2650 1950
 $Comp
-L +12C #PWR028
+L +12C #PWR19
 U 1 1 52493AD5
 P 2650 1250
-F 0 "#PWR028" H 2650 1220 30  0001 C CNN
+F 0 "#PWR19" H 2650 1220 30  0001 C CNN
 F 1 "+12C" H 2650 1360 40  0000 C CNN
 F 2 "" H 2650 1250 60  0000 C CNN
@@
 P 2950 1550
 F 0 "TH1" V 3050 1600 50  0000 C CNN
-F 1 "THERMISTOR" V 2850 1550 50  0000 C CNN
+F 1 "MINISMDC050F-2" V 2850 1550 50  0000 C CNN
 F 2 "~" H 2950 1550 60  0000 C CNN
 F 3 "~" H 2950 1550 60  0000 C CNN
+F 4 "TE Connectivity" H 2950 1550 60  0001 C CNN "MFG Name"
+F 5 "MINISMDC050F-2" H 2950 1550 60  0001 C CNN "MFG Part Number"
 	1    2950 1550
-	0    -1   -1   0
-$EndComp
-$Comp
-L THERMISTOR TH2
-U 1 1 52494037
-P 3350 1750
-F 0 "TH2" V 3450 1800 50  0000 C CNN
-F 1 "THERMISTOR" V 3250 1750 50  0000 C CNN
-F 2 "~" H 3350 1750 60  0000 C CNN
-F 3 "~" H 3350 1750 60  0000 C CNN
-	1    3350 1750
-	0    -1   -1   0
-$EndComp
-$Comp
-L THERMISTOR TH3
-U 1 1 5249403D
-P 3750 1950
-F 0 "TH3" V 3850 2000 50  0000 C CNN
-F 1 "THERMISTOR" V 3650 1950 50  0000 C CNN
-F 2 "~" H 3750 1950 60  0000 C CNN
-F 3 "~" H 3750 1950 60  0000 C CNN
-	1    3750 1950
-	0    -1   -1   0
-$EndComp
-$Comp
-L THERMISTOR TH4
-U 1 1 52494043
-P 4150 2150
-F 0 "TH4" V 4250 2200 50  0000 C CNN
-F 1 "THERMISTOR" V 4050 2150 50  0000 C CNN
-F 2 "~" H 4150 2150 60  0000 C CNN
-F 3 "~" H 4150 2150 60  0000 C CNN
-	1    4150 2150
 	0    -1   -1   0
 $EndComp
@@
 $EndComp
 $Comp
-L +5V #PWR029
+L +5V #PWR31
 U 1 1 525B1CA5
 P 6850 850
-F 0 "#PWR029" H 6850 940 20  0001 C CNN
+F 0 "#PWR31" H 6850 940 20  0001 C CNN
 F 1 "+5V" H 6850 940 30  0000 C CNN
 F 2 "" H 6850 850 60  0000 C CNN
@@
 $EndComp
 $Comp
-L GND #PWR030
+L GND #PWR30
 U 1 1 525B1CB4
 P 6400 1550
-F 0 "#PWR030" H 6400 1550 30  0001 C CNN
+F 0 "#PWR30" H 6400 1550 30  0001 C CNN
 F 1 "GND" H 6400 1480 30  0001 C CNN
 F 2 "" H 6400 1550 60  0000 C CNN
@@
 P 5900 1000
 F 0 "L4" V 5850 1000 40  0000 C CNN
-F 1 "INDUCTOR" V 6000 1000 40  0000 C CNN
+F 1 "CM322522-220KL" V 6000 1000 40  0000 C CNN
 F 2 "~" H 5900 1000 60  0000 C CNN
 F 3 "~" H 5900 1000 60  0000 C CNN
+F 4 "Bourns Inc" H 5900 1000 60  0001 C CNN "MFG Name"
+F 5 "CM322522-220KL" H 5900 1000 60  0001 C CNN "MFG Part Number"
 	1    5900 1000
 	0    -1   -1   0
@@
 	6400 1450 6400 1550
 $Comp
-L +3.3VP #PWR031
+L +3.3VP #PWR20
 U 1 1 525C49D8
 P 3300 1250
-F 0 "#PWR031" H 3350 1280 20  0001 C CNN
+F 0 "#PWR20" H 3350 1280 20  0001 C CNN
 F 1 "+3.3VP" H 3300 1340 30  0000 C CNN
 F 2 "" H 3300 1250 60  0000 C CNN
@@
 	1    0    0    -1
 $EndComp
+$Comp
+L THERMISTOR TH2
+U 1 1 5269F9D0
+P 3350 1750
+F 0 "TH2" V 3450 1650 50  0000 C CNN
+F 1 "MINISMDC050F-2" V 3250 1750 50  0000 C CNN
+F 2 "~" H 3350 1750 60  0000 C CNN
+F 3 "~" H 3350 1750 60  0000 C CNN
+F 4 "TE Connectivity" H 3350 1750 60  0001 C CNN "MFG Name"
+F 5 "MINISMDC050F-2" H 3350 1750 60  0001 C CNN "MFG Part Number"
+	1    3350 1750
+	0    -1   -1   0
+$EndComp
+$Comp
+L THERMISTOR TH3
+U 1 1 5269F9D8
+P 3750 1950
+F 0 "TH3" V 3850 1850 50  0000 C CNN
+F 1 "MINISMDC050F-2" V 3650 1950 50  0000 C CNN
+F 2 "~" H 3750 1950 60  0000 C CNN
+F 3 "~" H 3750 1950 60  0000 C CNN
+F 4 "TE Connectivity" H 3750 1950 60  0001 C CNN "MFG Name"
+F 5 "MINISMDC050F-2" H 3750 1950 60  0001 C CNN "MFG Part Number"
+	1    3750 1950
+	0    -1   -1   0
+$EndComp
+$Comp
+L THERMISTOR TH4
+U 1 1 5269F9E0
+P 4150 2150
+F 0 "TH4" V 4250 2050 50  0000 C CNN
+F 1 "MINISMDC050F-2" V 4050 2150 50  0000 C CNN
+F 2 "~" H 4150 2150 60  0000 C CNN
+F 3 "~" H 4150 2150 60  0000 C CNN
+F 4 "TE Connectivity" H 4150 2150 60  0001 C CNN "MFG Name"
+F 5 "MINISMDC050F-2" H 4150 2150 60  0001 C CNN "MFG Part Number"
+	1    4150 2150
+	0    -1   -1   0
+$EndComp
+$Comp
+L INDUCTOR L1
+U 1 1 5269FD5B
+P 5950 2050
+F 0 "L1" V 5900 2050 40  0000 C CNN
+F 1 "CM322522-220KL" V 6050 2050 40  0000 C CNN
+F 2 "~" H 5950 2050 60  0000 C CNN
+F 3 "~" H 5950 2050 60  0000 C CNN
+F 4 "Bourns Inc" H 5950 2050 60  0001 C CNN "MFG Name"
+F 5 "CM322522-220KL" H 5950 2050 60  0001 C CNN "MFG Part Number"
+	1    5950 2050
+	0    -1   -1   0
+$EndComp
+$Comp
+L INDUCTOR L2
+U 1 1 5269FD63
+P 5950 3150
+F 0 "L2" V 5900 3150 40  0000 C CNN
+F 1 "CM322522-220KL" V 6050 3150 40  0000 C CNN
+F 2 "~" H 5950 3150 60  0000 C CNN
+F 3 "~" H 5950 3150 60  0000 C CNN
+F 4 "Bourns Inc" H 5950 3150 60  0001 C CNN "MFG Name"
+F 5 "CM322522-220KL" H 5950 3150 60  0001 C CNN "MFG Part Number"
+	1    5950 3150
+	0    -1   1    0
+$EndComp
 $EndSCHEMATC
